Commit message: driving car with mesh

File: ros_ws/src/ackermann_vehicle_description/urdf/d.xacro (robot description, xacro)
@@ -32,9 +32,13 @@
   <xacro:property name="degrees_90" value="1.57079633"/>
   <!-- chassis_length is measured along the x axis, chassis_width
-       along the y axis, and chassis_height along the z axis. -->
+       along the y axis, and chassis_height along the z axis.
+  <xacro:property name="chassis_length" value="0.258"/>
+  <xacro:property name="chassis_width" value="0.168"/>
+  <xacro:property name="chassis_height" value="0.01"/>
+  <xacro:property name="chassis_mass" value="2.788"/> -->
   <xacro:property name="chassis_length" value="0.01"/>
   <xacro:property name="chassis_width" value="0.01"/>
-  <xacro:property name="chassis_height" value="0.01"/>
-  <xacro:property name="chassis_mass" value=".788"/>
+  <xacro:property name="chassis_height" value="0.5"/>
+  <xacro:property name="chassis_mass" value="2.788"/>
   <!-- battery_dist is the distance between the inner edges of the
        batteries. battery_comp_depth is the battery compartment depth.
@@ -58,25 +62,22 @@
   <xacro:property name="tire_width" value="0.0889"/>
   <xacro:property name="hex_hub_depth" value="0.01445"/>
-  <xacro:property name="wheel_mass" value="0.9"/>
- -->
-  <xacro:property name="hub_dia" value="0.005"/>
+  <xacro:property name="wheel_mass" value="0.29"/> -->
+  <xacro:property name="hub_dia" value="0.01"/>
   <xacro:property name="tire_dia" value="0.05"/>
-  <xacro:property name="tire_width" value="0.025"/>
-  <xacro:property name="hex_hub_depth" value="0.005"/>
-  <xacro:property name="wheel_mass" value="5"/>
+  <xacro:property name="tire_width" value="0.03"/>
+  <xacro:property name="hex_hub_depth" value="0.05"/>
+  <xacro:property name="wheel_mass" value="0.29"/>
   <!-- hex_hub_dist is the distance between left and right hex hubs when
        the shock absorbers are fully extended. axle_length is the distance
        from a U joint to the corresponding hex hub. wheel_travel is the
-       vertical wheel travel.
+       vertical wheel travel. -->
+  <xacro:property name="wheelbase" value="0.25"/>
+  <xacro:property name="hex_hub_dist" value="0.163"/>
+  <xacro:property name="axle_length" value="0.01"/>
+  <!--
   <xacro:property name="wheelbase" value="0.335"/>
-  <xacro:property name="hex_hub_dist" value="0.365"/>
-  <xacro:property name="axle_length" value="0.03"/>
+<xacro:property name="axle_length" value="0.03"/>
+      <xacro:property name="hex_hub_dist" value="0.365"/>-->
   <xacro:property name="wheel_travel" value="0.084"/>
-  <xacro:property name="shock_z_offset" value="0.0655"/>
- -->
-  <xacro:property name="wheelbase" value="0.22"/>
-  <xacro:property name="hex_hub_dist" value="0.153"/>
-  <xacro:property name="axle_length" value="0.0075"/>
-  <xacro:property name="wheel_travel" value="0.02"/>
   <xacro:property name="shock_z_offset" value="0.0655"/>
   <!-- shock_eff_limit is 2 * ((shock_stroke / 2) * shock_spring_constant) N.
@@ -102,8 +103,5 @@
   <!-- These constants are used to simulate a Traxxas 2056 servo operated at
        6 V. servo_stall_torque is measured in N m. servo_no_load_speed is
-       measured in rad/s.
-  <xacro:property name="servo_stall_torque" value="0.5649"/>
-  <xacro:property name="servo_no_load_speed" value="4.553"/>
--->
+       measured in rad/s. -->
   <xacro:property name="servo_stall_torque" value="0.5649"/>
   <xacro:property name="servo_no_load_speed" value="4.553"/>
@@ -155,4 +153,46 @@
                     outer_rad * outer_rad) / 2}"/>
     </inertial>
+  </xacro:macro>
+  <!-- Battery -->
+  <xacro:macro name="battery" params="prefix reflect">
+    <joint name="chassis_to_${prefix}_battery" type="fixed">
+      <parent link="chassis"/>
+      <child link="${prefix}_battery_offset"/>
+      <origin xyz="${battery_x_offset - battery_length / 2}
+                   ${reflect * battery_dist / 2}
+                   0"
+              rpy="${reflect * battery_comp_angle} 0 0"/>
+    </joint>
+    <link name="${prefix}_battery_offset">
+      <xacro:null_inertial/>
+    </link>
+    <joint name="offset_to_${prefix}_battery" type="fixed">
+      <parent link="${prefix}_battery_offset"/>
+      <child link="${prefix}_battery"/>
+      <origin xyz="0
+                   ${reflect * battery_width / 2}
+                   ${(battery_height / 2) - battery_comp_depth}"/>
+    </joint>
+    <link name="${prefix}_battery">
+	<visual>
+        <geometry>
+          <box size="${battery_length} ${battery_width} ${battery_height}"/>
+        </geometry>
+        <material name="battery_mat"/>
+      </visual>
+      <collision>
+        <geometry>
+          <box size="${battery_length} ${battery_width} ${battery_height}"/>
+        </geometry>
+      </collision>
+      <xacro:solid_cuboid_inertial
+         width="${battery_length}" depth="${battery_width}"
+         height="${battery_height}" mass="${battery_mass}">
+        <origin/>
+      </xacro:solid_cuboid_inertial>
+    </link>
+    <gazebo reference="${prefix}_battery">
+      <material>Gazebo/Blue</material>
+    </gazebo>
   </xacro:macro>
   <!-- Shock absorber -->
@@ -233,5 +273,5 @@
     </link>
     <gazebo reference="${lr_prefix}_${fr_prefix}_wheel">
-      <material>Gazebo/Gold</material>
+      <material>Gazebo/Black</material>
     </gazebo>
   </xacro:macro>
@@ -279,5 +319,4 @@
        rviz. -->
   <link name="base_link">
-<!--
     <visual>
       <geometry>
@@ -286,5 +325,4 @@
       <material name="chassis_mat"/>
     </visual>
--->
   </link>
   <gazebo reference="base_link">
@@ -295,5 +333,5 @@
 <!--
     <visual>
-      <origin xyz="0 0 ${-chassis_height / 2}"/>
+      <origin xyz="0 0 ${chassis_height / 2}"/>
       <geometry>
         <box size="${chassis_length} ${chassis_width} ${chassis_height}"/>
@@ -302,5 +340,5 @@
     </visual>
     <collision>
-      <origin xyz="0 0 ${-chassis_height / 2}"/>
+      <origin xyz="0 0 ${chassis_height / 2}"/>
       <geometry>
         <box size="${chassis_length} ${chassis_width} ${chassis_height}"/>
@@ -308,14 +346,8 @@
     </collision>
 -->
-        <visual name="visual">
-	  <origin xyz="0.15 -0.09 -0.09" rpy="0 0 ${degrees_90}" />
-          <geometry>
-  	    <mesh filename="package://ackermann_vehicle_description/meshes/car_black.dae" scale="1 1 1"/>
-          </geometry>
-        </visual>
     <xacro:solid_cuboid_inertial
         width="${chassis_length}" depth="${chassis_width}"
         height="${chassis_height}" mass="${chassis_mass}">
-      <origin xyz="0 0 ${-chassis_height / 2}"/>
+      <origin xyz="0 0 ${chassis_height / 2}"/>
     </xacro:solid_cuboid_inertial>
   </link>
